File: KiCad files/Psion Organiser II XP Issue3 Power PCB.sch (KiCad schematic (older format))
At the start: 76 parts, among them U1 74LS132, X1 LM324

Commit message: tidied up schematic
Parts:
- gave numbers to parts that had none: 1
Other:
- note added: "Semi-custom logic IC clock moved\nfrom mainboard at Issue 3 PCB"
- note added: "Vcc1 regulator\nMainboard \nsupply"
- note removed: "Clock moved from mainboard\nat Issue 3 PCB"
- note removed: "Vcc1 regulator\nMainboard supply"
- moved on the sheet: C1, C10?, C11, C12, C13, C14, C15, C7, C8, C9?, D3A, D3B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

Commit message: slight mod
Parts:
- gave numbers to parts that had none: 1
Other:
- moved on the sheet: R18?
Changed lines of the file:
@@
 Wire Wire Line
 	9550 2200 9700 2200
-$Comp
-L Device:R R5
-U 1 1 613E9641
-P 8000 2600
-F 0 "R5" H 8070 2646 50  0000 L CNN
-F 1 "510K" H 8070 2555 50  0000 L CNN
-F 2 "" V 7930 2600 50  0001 C CNN
-F 3 "~" H 8000 2600 50  0001 C CNN
-	1    8000 2600
-	1    0    0    -1
-$EndComp
 Wire Wire Line
 	8000 2850 8000 2800
-Wire Wire Line
-	8000 2200 8000 2450
 Wire Wire Line
 	7500 3650 7500 3250
 Connection ~ 8000 2800
-Wire Wire Line
-	8000 2800 8000 2750
 $Comp
 L Device:Q_NPN_BCE TR2
@@
 $EndComp
 $Comp
-L Device:R R19?
+L Device:R R18?
 U 1 1 615591E8
-P 10150 7950
-F 0 "R19?" H 10220 7996 50  0000 L CNN
-F 1 "47K" H 10220 7905 50  0000 L CNN
-F 2 "" V 10080 7950 50  0001 C CNN
-F 3 "~" H 10150 7950 50  0001 C CNN
-	1    10150 7950
-	1    0    0    -1
-$EndComp
-Wire Wire Line
-	10150 7800 10150 2200
+P 10150 7800
+F 0 "R18?" H 10220 7846 50  0000 L CNN
+F 1 "47K" H 10220 7755 50  0000 L CNN
+F 2 "" V 10080 7800 50  0001 C CNN
+F 3 "~" H 10150 7800 50  0001 C CNN
+	1    10150 7800
+	1    0    0    -1
+$EndComp
+Wire Wire Line
+	10150 7650 10150 2200
 Connection ~ 10150 2200
 Wire Wire Line
@@
 Wire Notes Line
 	11800 6900 10850 6900
-Connection ~ 10150 8100
-Wire Wire Line
-	10150 8100 10350 8100
 $Comp
 L Connector:Conn_01x27_Female Mainboard
@@
 F 2 "" H 2438 5950 50  0001 C CNN
 F 3 "~" H 2400 6100 50  0001 C CNN
-F 4 "30 V" H 2550 5950 50  0000 L CNN "Max Voltage"
+F 4 "30 V" H 2650 6100 50  0000 L CNN "Max Voltage"
 	1    2400 6100
 	1    0    0    -1
@@
 Wire Wire Line
 	14300 6800 15000 6800
-Wire Wire Line
-	5950 8100 10150 8100
 Text Notes 1200 5100 0    79   ~ 0
 1024 Hz
@@
 Wire Wire Line
 	6800 3750 5950 3750
-Text Notes 15050 2500 0    59   ~ 0
+Text Notes 15000 2500 0    59   ~ 0
 pullup
 Text Notes 14900 850  0    59   ~ 0
@@
 	-1   0    0    -1
 $EndComp
+Wire Wire Line
+	10150 2200 10150 2050
+Wire Wire Line
+	5950 8100 10150 8100
+Wire Wire Line
+	10150 7950 10150 8100
+Connection ~ 10150 8100
+Wire Wire Line
+	10150 8100 10350 8100
+Wire Wire Line
+	8000 2800 8000 2750
+Wire Wire Line
+	8000 2200 8000 2450
+$Comp
+L Device:R R5
+U 1 1 613E9641
+P 8000 2600
+F 0 "R5" H 8070 2646 50  0000 L CNN
+F 1 "510K" H 8070 2555 50  0000 L CNN
+F 2 "" V 7930 2600 50  0001 C CNN
+F 3 "~" H 8000 2600 50  0001 C CNN
+	1    8000 2600
+	1    0    0    -1
+$EndComp
 $EndSCHEMATC

Commit message: tidy up
Changed lines of the file:
@@
 $EndComp
-Wire Wire Line
-	10150 2200 10150 2050
 Wire Wire Line
 	5950 8100 10150 8100
